Commit message: Added IMU simulation. Removed pillar links.

File: mecabot_body/urdf/chassis/layer.xacro (robot description, xacro)
@@ -19,5 +19,5 @@
         </visual>
     </xacro:macro>
-    <xacro:macro name="direction_pieces">
+    <xacro:macro name="direction_pieces_visual">
         <visual name="direction_piece_1">
             <origin xyz="${length/2-side_piece_size/2} 0.0 ${height/2}" rpy="0.0 0.0 0.0"/>
@@ -48,4 +48,15 @@
         </visual>
     </xacro:macro>
+    <xacro:macro name="pillar_visual" params="side_FB side_LR">
+        <visual>
+            <origin xyz="${pillar_offset_fb*side_FB} ${pillar_offset_lr*side_LR} ${-pillar_length/2}" rpy="0.0 0.0 0.0"/>
+            <geometry>
+                <cylinder radius="${pillar_radius}" length="${pillar_length}"/>
+            </geometry>
+            <material name="pillar_color">
+                <color rgba="${255/255} ${108/255} ${12/255} 1.0"/>
+            </material>
+        </visual>
+    </xacro:macro>
     <xacro:macro name="layer" params="name parent mass length width height reflect">
         <xacro:property name="layer_joint_origin">
@@ -61,5 +72,11 @@
             </visual>
             <xacro:if value="${name == 'upper_layer'}">
-                <xacro:direction_pieces/>
+                <xacro:direction_pieces_visual/>
+                <xacro:pillar_visual side_FB="1" side_LR="0"/>
+                <xacro:pillar_visual side_FB="1" side_LR="1"/>
+                <xacro:pillar_visual side_FB="1" side_LR="-1"/>
+                <xacro:pillar_visual side_FB="-1" side_LR="0"/>
+                <xacro:pillar_visual side_FB="-1" side_LR="1"/>
+                <xacro:pillar_visual side_FB="-1" side_LR="-1"/>
             </xacro:if>
             <xacro:if value="${name == 'lower_layer'}">

File: mecabot_body/urdf/include/common_macros.xacro (robot description, xacro)
@@ -48,5 +48,4 @@
     <xacro:property name="pillar_radius" value="0.002"/>
     <xacro:property name="pillar_length" value="0.055"/>
-    <xacro:property name="pillar_mass" value="0.005"/>
     <xacro:property name="pillar_offset_fb" value="0.12"/>
     <xacro:property name="pillar_offset_lr" value="0.055"/>

File: mecabot_body/urdf/mecabot.urdf.xacro (robot description, xacro)
@@ -1,4 +1,5 @@
 <?xml version="1.0"?>
 <robot xmlns:xacro="http://www.ros.org/wiki/xacro" name="mecabot">
-    <xacro:include filename="mecabot_core.xacro"/>
+    <xacro:include filename="$(find mecabot_body)/urdf/mecabot_core.xacro"/>
+    <!-- <xacro:include filename="$(find mecabot_body)/urdf/gazebo_control.xacro"/> -->
 </robot>

File: mecabot_body/urdf/mecabot_core.xacro (robot description, xacro)
@@ -3,10 +3,9 @@
     <xacro:include filename="$(find mecabot_body)/urdf/include/common_macros.xacro"/>
     <xacro:include filename="$(find mecabot_body)/urdf/include/materials.xacro"/>
-    <xacro:include filename="$(find mecabot_body)/urdf/chassis/pillar.xacro"/>
     <xacro:include filename="$(find mecabot_body)/urdf/chassis/layer.xacro"/>
     <xacro:include filename="$(find mecabot_body)/urdf/wheels/wheel.xacro"/>
     <xacro:include filename="$(find mecabot_body)/urdf/wheels/mecanum_wheel.xacro"/>
+    <xacro:include filename="$(find mecabot_body)/urdf/sensors/imu.xacro"/>
     <xacro:include filename="$(find mecabot_body)/urdf/sensors/lidar.xacro"/>
-    <xacro:include filename="$(find mecabot_body)/urdf/mecabot.gazebo.xacro"/>
     <!--~~~~~~~~~~ BASE LINK ~~~~~~~~~~-->
     <link name="base_link">
@@ -18,19 +17,7 @@
         </collision>
     </link>
-    <!--~~~~~~~~~~ LAYER AND PILLAR LINKS ~~~~~~~~~~-->
+    <!--~~~~~~~~~~ CHASSIS LAYERS ~~~~~~~~~~-->
     <xacro:layer name="lower_layer" parent="base" mass="${layer_mass}"
                 length="${layer_l}" width="${layer_w-wheel_thickness*2}" height="${layer_h}" reflect="0"/>
-    <xacro:pillar name="one" parent="base" mass="${pillar_mass}"
-                radius="${pillar_radius}" length="${pillar_length}" side_FB="1" side_LR="0"/>
-    <xacro:pillar name="two" parent="base" mass="${pillar_mass}"
-                radius="${pillar_radius}" length="${pillar_length}" side_FB="1" side_LR="1"/>
-    <xacro:pillar name="three" parent="base" mass="${pillar_mass}"
-                 radius="${pillar_radius}" length="${pillar_length}" side_FB="1" side_LR="-1"/>
-    <xacro:pillar name="four" parent="base" mass="${pillar_mass}"
-                radius="${pillar_radius}" length="${pillar_length}" side_FB="-1" side_LR="0"/>
-    <xacro:pillar name="five" parent="base" mass="${pillar_mass}"
-                radius="${pillar_radius}" length="${pillar_length}" side_FB="-1" side_LR="1"/>
-    <xacro:pillar name="six" parent="base" mass="${pillar_mass}"
-                radius="${pillar_radius}" length="${pillar_length}" side_FB="-1" side_LR="-1"/>
     <xacro:layer name="upper_layer" parent="base" mass="${layer_mass}"
                 length="${layer_l}" width="${layer_w-wheel_thickness*2}" height="${layer_h}" reflect="1"/>
@@ -46,9 +33,16 @@
     <!--~~~~~~~~~~ LIDAR ~~~~~~~~~~-->
     <xacro:lidar parent="upper_layer"/>
-    <gazebo>
+    <!--~~~~~~~~~~ IMU ~~~~~~~~~~-->
+    <xacro:imu parent="lower_layer"/>
+    <!-- <gazebo>
         <plugin name="joint_state_publisher" filename="libgazebo_ros_joint_state_publisher.so">
             <jointName>front_left_wheel_joint, front_right_wheel_joint, back_left_wheel_joint, back_right_wheel_joint</jointName>
         </plugin>
+    </gazebo> -->
+    <!--~~~~~~~~~~ ros_control ~~~~~~~~~~-->
+    <gazebo>
+        <plugin name="gazebo_ros_control" filename="libgazebo_ros_control.so">
+            <robotNamespace>/mecabot</robotNamespace>
+        </plugin>
     </gazebo>
-    <xacro:mecanum_drive/>
 </robot>

File: mecabot_body/urdf/sensors/lidar.xacro (robot description, xacro)
@@ -32,5 +32,5 @@
                 <pose> 0 0 0 0 0 0 </pose>
                 <visualize>true</visualize>
-                <update_rate>10</update_rate>
+                <update_rate>30</update_rate>
                 <ray>
                     <scan>
@@ -45,10 +45,17 @@
                         <min>0.2</min>
                         <max>12</max>
+                        <resolution>0.01</resolution>
                     </range>
+                    <noise>
+                        <type>gaussian</type>
+                        <mean>0.0</mean>
+                        <stddev>0.01</stddev>
+                    </noise>
                 </ray>
                 <plugin name="laser_controller" filename="libgazebo_ros_laser.so">
+                    <robotNamespace></robotNamespace>
                     <topicName>/mecabot/laser/scan</topicName>
                     <frameName>lidar_frame</frameName>
-                  </plugin>
+                </plugin>
             </sensor>
         </gazebo>

File: mecabot_body/urdf/wheels/wheel.xacro (robot description, xacro)
@@ -32,4 +32,14 @@
             <dynamic damping="0.01" friction="0.0"/>
         </joint>
+        <transmission name="${name}_wheel_transmission">
+            <type>transmission_interface/SimpleTransmission</type>
+            <joint name="${name}_wheel_joint">
+                <hardwareInterface>hardware_interface/EffortJointInterface</hardwareInterface>
+            </joint>
+            <actuator name="{name}_motor">
+                <mechanicalReduction>1.0</mechanicalReduction>
+                <hardwareInterface>hardware_interface/EffortJointInterface</hardwareInterface>
+            </actuator>
+        </transmission>
         <gazebo reference="${name}_wheel_link">
             <material>Gazebo/Yellow</material>
