Commit message: Added ros_control plugin.

File: mecabot_body/urdf/mecabot_core.xacro (robot description, xacro)
@@ -17,4 +17,5 @@
         </collision>
     </link>
+    <!-- Fix the cobot to the world-->
     <!--~~~~~~~~~~ CHASSIS LAYERS ~~~~~~~~~~-->
     <xacro:layer name="lower_layer" parent="base" mass="${layer_mass}"
@@ -32,7 +33,7 @@
                 radius="${wheel_radius}" thickness="${wheel_thickness}" side_FB="-1" side_LR="-1"/>
     <!--~~~~~~~~~~ LIDAR ~~~~~~~~~~-->
-    <xacro:lidar parent="upper_layer"/>
+    <!-- <xacro:lidar parent="upper_layer"/>  -->
     <!--~~~~~~~~~~ IMU ~~~~~~~~~~-->
-    <xacro:imu parent="lower_layer"/>
+    <xacro:imu parent="base"/>
     <!-- <gazebo>
         <plugin name="joint_state_publisher" filename="libgazebo_ros_joint_state_publisher.so">

File: mecabot_body/urdf/sensors/imu.xacro (robot description, xacro)
@@ -29,4 +29,5 @@
                 <topic>__default_topic__</topic>
                 <plugin name="imu_plugin" filename="libgazebo_ros_imu_sensor.so">
+                    <robotNamespace>/mecabot</robotNamespace>
                     <topicName>imu</topicName>
                     <bodyName>imu_frame</bodyName>

File: mecabot_body/urdf/wheels/wheel.xacro (robot description, xacro)
@@ -2,7 +2,4 @@
 <robot xmlns:xacro="http://www.ros.org/wiki/xacro">
     <xacro:macro name="wheel" params="name parent mass radius thickness side_FB side_LR">
-        <xacro:property name="wheel_joint_origin">
-            <origin xyz="${wheel_offset_fb*side_FB} ${wheel_offset_lr*side_LR} -${wheel_offset_z}" rpy="${-side_LR*PI/2} 0.0 0.0"/>
-        </xacro:property>
         <link name="${name}_wheel_link">
             <visual>
@@ -28,5 +25,5 @@
             <parent link="${parent}_link"/>
             <child link="${name}_wheel_link"/>
-            <xacro:insert_block name="wheel_joint_origin" />
+            <origin xyz="${wheel_offset_fb*side_FB} ${wheel_offset_lr*side_LR} -${wheel_offset_z}" rpy="${-side_LR*PI/2} 0.0 0.0"/>
             <axis xyz="0 0 ${side_LR}" rpy="0 0 0" />
             <dynamic damping="0.01" friction="0.0"/>
@@ -37,5 +34,5 @@
                 <hardwareInterface>hardware_interface/EffortJointInterface</hardwareInterface>
             </joint>
-            <actuator name="{name}_motor">
+            <actuator name="${name}_motor">
                 <mechanicalReduction>1.0</mechanicalReduction>
                 <hardwareInterface>hardware_interface/EffortJointInterface</hardwareInterface>
