Commit message: Added World spawn file. Changed workspace structure.

File: mecabot_body/urdf/gazebo_control.xacro (robot description, xacro)
@@ -2,21 +2,12 @@
 <robot xmlns:xacro="http://www.ros.org/wiki/xacro">
     <gazebo>
-        <plugin name="skid_steer_drive_controller" filename="libgazebo_ros_skid_steer_drive.so">
-            <updateRate>100.0</updateRate>
+        <plugin name="mecabot_controller" filename="libgazebo_ros_planar_move.so">
             <robotNamespace>/</robotNamespace>
-            <leftFrontJoint>front_left_wheel_joint</leftFrontJoint>
-            <rightFrontJoint>front_right_wheel_joint</rightFrontJoint>
-            <leftRearJoint>rear_left_wheel_joint</leftRearJoint>
-            <rightRearJoint>rear_right_wheel_joint</rightRearJoint>
-            <wheelSeparation>0.12</wheelSeparation>
-            <wheelDiameter>0.06</wheelDiameter>
-            <torque>10</torque>
             <commandTopic>cmd_vel</commandTopic>
             <odometryTopic>odom</odometryTopic>
             <odometryFrame>odom</odometryFrame>
+            <odometryRate>20.0</odometryRate>
             <robotBaseFrame>base_link</robotBaseFrame>
-            <publishWheelTF>true</publishWheelTF>
-            <publishOdom>true</publishOdom>
-            <publishWheelJointState>true</publishWheelJointState>
+            <publishTF>true</publishTF>
         </plugin>
     </gazebo>

File: mecabot_body/urdf/include/common_macros.xacro (robot description, xacro)
@@ -25,5 +25,5 @@
     <xacro:property name="layer_w" value="0.15"/>
     <xacro:property name="layer_h" value="0.002"/>
-    <xacro:property name="layer_mass" value="0.07"/>
+    <xacro:property name="layer_mass" value="1.0"/>
     <xacro:property name="side_piece_size" value="0.03"/>
     <xacro:property name="motor_l" value="0.07"/>
@@ -41,5 +41,5 @@
     <xacro:property name="wheel_radius" value="0.03" />
     <xacro:property name="wheel_thickness" value="0.031" />
-    <xacro:property name="wheel_mass" value="0.04" /> <!-- in kg-->
+    <xacro:property name="wheel_mass" value="0.5" /> <!-- in kg-->
     <xacro:property name="wheel_offset_z" value="0.009" />
     <xacro:property name="wheel_offset_fb" value="0.06215"/>

File: mecabot_body/urdf/mecabot.urdf.xacro (robot description, xacro)
@@ -2,4 +2,4 @@
 <robot xmlns:xacro="http://www.ros.org/wiki/xacro" name="mecabot">
     <xacro:include filename="$(find mecabot_body)/urdf/mecabot_core.xacro"/>
-    <!-- <xacro:include filename="$(find mecabot_body)/urdf/gazebo_control.xacro"/> -->
+    <xacro:include filename="$(find mecabot_body)/urdf/gazebo_control.xacro"/>
 </robot>

File: mecabot_body/urdf/mecabot_core.xacro (robot description, xacro)
@@ -10,12 +10,5 @@
     <!--~~~~~~~~~~ BASE LINK ~~~~~~~~~~-->
     <link name="base_link">
-        <collision>
-            <origin xyz="0.0 0.0 ${chassis_h/2}" rpy="0.0 0.0 0.0"/>
-            <geometry>
-                <box size="${chassis_l} ${chassis_w} ${chassis_h}"/>
-            </geometry>
-        </collision>
     </link>
-    <!-- Fix the cobot to the world-->
     <!--~~~~~~~~~~ CHASSIS LAYERS ~~~~~~~~~~-->
     <xacro:layer name="lower_layer" parent="base" mass="${layer_mass}"
@@ -33,17 +26,17 @@
                 radius="${wheel_radius}" thickness="${wheel_thickness}" side_FB="-1" side_LR="-1"/>
     <!--~~~~~~~~~~ LIDAR ~~~~~~~~~~-->
-    <!-- <xacro:lidar parent="upper_layer"/>  -->
+    <xacro:lidar parent="upper_layer"/>
     <!--~~~~~~~~~~ IMU ~~~~~~~~~~-->
     <xacro:imu parent="base"/>
-    <!-- <gazebo>
+    <gazebo>
         <plugin name="joint_state_publisher" filename="libgazebo_ros_joint_state_publisher.so">
             <jointName>front_left_wheel_joint, front_right_wheel_joint, back_left_wheel_joint, back_right_wheel_joint</jointName>
         </plugin>
-    </gazebo> -->
+    </gazebo>
     <!--~~~~~~~~~~ ros_control ~~~~~~~~~~-->
-    <gazebo>
+    <!-- <gazebo>
         <plugin name="gazebo_ros_control" filename="libgazebo_ros_control.so">
             <robotNamespace>/mecabot</robotNamespace>
         </plugin>
-    </gazebo>
+    </gazebo> -->
 </robot>

File: mecabot_body/urdf/sensors/lidar.xacro (robot description, xacro)
@@ -36,5 +36,5 @@
                     <scan>
                         <horizontal>
-                            <samples>360</samples>
+                            <samples>359</samples>
                             <resolution>1</resolution>
                             <min_angle>-3.14</min_angle>
@@ -50,10 +50,10 @@
                         <type>gaussian</type>
                         <mean>0.0</mean>
-                        <stddev>0.01</stddev>
+                        <stddev>0.02</stddev>
                     </noise>
                 </ray>
                 <plugin name="laser_controller" filename="libgazebo_ros_laser.so">
-                    <robotNamespace></robotNamespace>
-                    <topicName>/mecabot/laser/scan</topicName>
+                    <robotNamespace>/mecabot</robotNamespace>
+                    <topicName>/laser/scan</topicName>
                     <frameName>lidar_frame</frameName>
                 </plugin>

File: mecabot_body/urdf/wheels/mecanum_wheel.xacro (robot description, xacro)
@@ -34,4 +34,6 @@
             </visual>
             <collision>
+                <mu1>0.3</mu1>
+                <mu2>0.3</mu2>
                 <origin xyz="0 0 0" rpy="0 0 0" />
                 <geometry>

File: mecabot_body/urdf/wheels/wheel.xacro (robot description, xacro)
@@ -22,4 +22,11 @@
             </xacro:inertial_cylinder>
         </link>
+        <gazebo reference="${name}_wheel_link">
+			<mu1 value="0.5"/>
+			<mu2 value="0.5"/>
+			<kp value="10000000.0" />
+			<kd value="1.0" />
+			<fdir1 value="1 0 0"/>
+		</gazebo>
         <joint name="${name}_wheel_joint" type="continuous">
             <parent link="${parent}_link"/>
@@ -27,7 +34,6 @@
             <origin xyz="${wheel_offset_fb*side_FB} ${wheel_offset_lr*side_LR} -${wheel_offset_z}" rpy="${-side_LR*PI/2} 0.0 0.0"/>
             <axis xyz="0 0 ${side_LR}" rpy="0 0 0" />
-            <dynamic damping="0.01" friction="0.0"/>
         </joint>
-        <transmission name="${name}_wheel_transmission">
+        <!-- <transmission name="${name}_wheel_transmission">
             <type>transmission_interface/SimpleTransmission</type>
             <joint name="${name}_wheel_joint">
@@ -38,5 +44,5 @@
                 <hardwareInterface>hardware_interface/EffortJointInterface</hardwareInterface>
             </actuator>
-        </transmission>
+        </transmission> -->
         <gazebo reference="${name}_wheel_link">
             <material>Gazebo/Yellow</material>
