Commit message: Fixed gazebo simulation.

File: mecabot_description/urdf/mecabot.urdf.xacro (robot description, xacro)
@@ -1,5 +1,5 @@
 <?xml version="1.0"?>
 <robot xmlns:xacro="http://www.ros.org/wiki/xacro" name="mecabot">
-    <xacro:include filename="$(find mecabot_description)/urdf/mecabot_core.xacro"/>
+    <xacro:include filename="$(find mecabot_description)/urdf/mecabot_core.xacro" />
     <xacro:include filename="$(find mecabot_description)/urdf/gazebo_control.xacro"/>
 </robot>

File: mecabot_description/urdf/mecabot_core.xacro (robot description, xacro)
@@ -1,5 +1,5 @@
 <?xml version="1.0"?>
 <robot xmlns:xacro="http://www.ros.org/wiki/xacro">
-    <xacro:property name="simulation" value="false"/>
+    <xacro:arg name="use_simulation" default="false"/>
     <xacro:include filename="$(find mecabot_description)/urdf/include/common_macros.xacro"/>
     <xacro:include filename="$(find mecabot_description)/urdf/include/materials.xacro"/>
@@ -31,5 +31,5 @@
     <xacro:imu parent="base"/>
     <!--~~~~~~~~~~ Extra simulation components (if use Gazebo). Change condition to False when run on real robot  ~~~~~~~~~~-->
-    <xacro:if value="${simulation == 'true'}">
+    <xacro:if value="$(arg use_simulation)">
         <!-- Publish joints' state -->
         <gazebo>
