Commit message: Created teleop package for manual driving. Added comments.

File: mecabot_description/urdf/mecabot_core.xacro (robot description, xacro)
@@ -1,4 +1,5 @@
 <?xml version="1.0"?>
 <robot xmlns:xacro="http://www.ros.org/wiki/xacro">
+    <xacro:property name="simulation" value="false"/>
     <xacro:include filename="$(find mecabot_description)/urdf/include/common_macros.xacro"/>
     <xacro:include filename="$(find mecabot_description)/urdf/include/materials.xacro"/>
@@ -28,15 +29,69 @@
     <xacro:lidar parent="upper_layer"/>
     <!--~~~~~~~~~~ IMU ~~~~~~~~~~-->
-    <!-- <xacro:imu parent="base"/> -->
-    <gazebo>
-        <plugin name="joint_state_publisher" filename="libgazebo_ros_joint_state_publisher.so">
-            <jointName>front_left_wheel_joint, front_right_wheel_joint, back_left_wheel_joint, back_right_wheel_joint</jointName>
-        </plugin>
-    </gazebo>
-    <!--~~~~~~~~~~ ros_control ~~~~~~~~~~-->
-    <!-- <gazebo>
-        <plugin name="gazebo_ros_control" filename="libgazebo_ros_control.so">
-            <robotNamespace>/mecabot</robotNamespace>
-        </plugin>
-    </gazebo> -->
+    <xacro:imu parent="base"/>
+    <!--~~~~~~~~~~ Extra simulation components (if use Gazebo). Change condition to False when run on real robot  ~~~~~~~~~~-->
+    <xacro:if value="${simulation == 'true'}">
+        <!-- Publish joints' state -->
+        <gazebo>
+            <plugin name="joint_state_publisher" filename="libgazebo_ros_joint_state_publisher.so">
+                <jointName>front_left_wheel_joint, front_right_wheel_joint, back_left_wheel_joint, back_right_wheel_joint</jointName>
+            </plugin>
+        </gazebo>
+        <!-- Lidar simulation using Gazebo. -->
+        <gazebo reference="lidar_frame">
+            <material>Gazebo/Black</material>
+            <sensor name="laser" type="ray">
+                <pose> 0 0 0 0 0 0 </pose>
+                <visualize>true</visualize>
+                <update_rate>30</update_rate>
+                <ray>
+                    <scan>
+                        <horizontal>
+                            <samples>359</samples>
+                            <resolution>1</resolution>
+                            <min_angle>-3.14</min_angle>
+                            <max_angle>3.14</max_angle>
+                        </horizontal>
+                    </scan>
+                    <range>
+                        <min>0.2</min>
+                        <max>12</max>
+                        <resolution>0.01</resolution>
+                    </range>
+                    <noise>
+                        <type>gaussian</type>
+                        <mean>0.0</mean>
+                        <stddev>0.02</stddev>
+                    </noise>
+                </ray>
+                <plugin name="laser_controller" filename="libgazebo_ros_laser.so">
+                    <robotNamespace>/</robotNamespace>
+                    <topicName>/scan</topicName>
+                    <frameName>lidar_frame</frameName>
+                </plugin>
+            </sensor>
+        </gazebo>
+        <!-- IMU simulation using Gazebo. -->
+        <gazebo reference="imu_frame">
+            <gravity>true</gravity>
+            <sensor name="imu_sensor" type="imu">
+                <always_on>true</always_on>
+                <update_rate>100</update_rate>
+                <visualize>true</visualize>
+                <topic>__default_topic__</topic>
+                <plugin name="imu_plugin" filename="libgazebo_ros_imu_sensor.so">
+                    <robotNamespace>/</robotNamespace>
+                    <topicName>/imu</topicName>
+                    <bodyName>imu_frame</bodyName>
+                    <updateRateHZ>10.0</updateRateHZ>
+                    <gaussianNoise>0.0</gaussianNoise>
+                    <xyzOffset>0 0 0</xyzOffset>
+                    <rpyOffset>0 0 0</rpyOffset>
+                    <frameName>imu_frame</frameName>
+                    <initialOrientationAsReference>false</initialOrientationAsReference>
+                </plugin>
+                <pose>0 0 0 0 0 0</pose>
+            </sensor>
+        </gazebo>
+    </xacro:if>
 </robot>

File: mecabot_description/urdf/sensors/imu.xacro (robot description, xacro)
@@ -2,5 +2,5 @@
 <robot xmlns:xacro="http://www.ros.org/wiki/xacro">
     <xacro:macro name="imu" params="parent">
-        <joint name="joint_name" type="fixed">
+        <joint name="imu_joint" type="fixed">
             <origin xyz="0.0 0.0 0.0" rpy="0.0 0.0 0.0"/>
             <parent link="${parent}_link"/>
@@ -21,25 +21,4 @@
             </collision>
         </link>
-        <gazebo reference="imu_frame">
-            <gravity>true</gravity>
-            <sensor name="imu_sensor" type="imu">
-                <always_on>true</always_on>
-                <update_rate>100</update_rate>
-                <visualize>true</visualize>
-                <topic>__default_topic__</topic>
-                <plugin name="imu_plugin" filename="libgazebo_ros_imu_sensor.so">
-                    <robotNamespace>/mecabot</robotNamespace>
-                    <topicName>imu</topicName>
-                    <bodyName>imu_frame</bodyName>
-                    <updateRateHZ>10.0</updateRateHZ>
-                    <gaussianNoise>0.0</gaussianNoise>
-                    <xyzOffset>0 0 0</xyzOffset>
-                    <rpyOffset>0 0 0</rpyOffset>
-                    <frameName>imu_frame</frameName>
-                    <initialOrientationAsReference>false</initialOrientationAsReference>
-                </plugin>
-                <pose>0 0 0 0 0 0</pose>
-            </sensor>
-        </gazebo>
     </xacro:macro>
 </robot>

File: mecabot_description/urdf/sensors/lidar.xacro (robot description, xacro)
@@ -27,38 +27,4 @@
             </xacro:inertial_cylinder>
         </link>
-        <!-- Lidar simulation using Gazebo. Change condition to False when run on real robot -->
-        <gazebo reference="lidar_frame">
-            <material>Gazebo/Black</material>
-            <sensor name="laser" type="ray">
-                <pose> 0 0 0 0 0 0 </pose>
-                <visualize>true</visualize>
-                <update_rate>30</update_rate>
-                <ray>
-                    <scan>
-                        <horizontal>
-                            <samples>359</samples>
-                            <resolution>1</resolution>
-                            <min_angle>-3.14</min_angle>
-                            <max_angle>3.14</max_angle>
-                        </horizontal>
-                    </scan>
-                    <range>
-                        <min>0.2</min>
-                        <max>12</max>
-                        <resolution>0.01</resolution>
-                    </range>
-                    <noise>
-                        <type>gaussian</type>
-                        <mean>0.0</mean>
-                        <stddev>0.02</stddev>
-                    </noise>
-                </ray>
-                <plugin name="laser_controller" filename="libgazebo_ros_laser.so">
-                    <robotNamespace>/</robotNamespace>
-                    <topicName>/scan</topicName>
-                    <frameName>lidar_frame</frameName>
-                </plugin>
-            </sensor>
-        </gazebo>
     </xacro:macro>
 </robot>

Commit message: Somehow it kinda work now.

File: mecabot_description/urdf/mecabot_core.xacro (robot description, xacro)
@@ -27,7 +27,7 @@
                 radius="${wheel_radius}" thickness="${wheel_thickness}" side_FB="-1" side_LR="-1"/>
     <!--~~~~~~~~~~ LIDAR ~~~~~~~~~~-->
-    <xacro:lidar parent="upper_layer"/>
+    <xacro:lidar parent="base"/>
     <!--~~~~~~~~~~ IMU ~~~~~~~~~~-->
-    <xacro:imu parent="upper_layer"/>
+    <xacro:imu parent="base"/>
     <!--~~~~~~~~~~ Extra simulation components (if use Gazebo). Change condition to False when run on real robot  ~~~~~~~~~~-->
     <xacro:if value="$(arg use_simulation)">

File: mecabot_description/urdf/sensors/imu.xacro (robot description, xacro)
@@ -3,5 +3,5 @@
     <xacro:macro name="imu" params="parent">
         <joint name="imu_joint" type="fixed">
-            <origin xyz="-0.1065 0.0 0.0" rpy="0.0 0.0 0.0"/>
+            <origin xyz="-0.1065 0.0 0.072" rpy="0.0 0.0 0.0"/>
             <parent link="${parent}_link"/>
             <child link="imu_frame"/>

File: mecabot_description/urdf/sensors/lidar.xacro (robot description, xacro)
@@ -3,5 +3,5 @@
     <xacro:macro name="lidar" params="parent">
         <xacro:property name="lidar_joint_origin">
-            <origin xyz="0 0 ${lidar_height/2}" rpy="0.0 0.0 0.0"/>
+            <origin xyz="0 0 ${lidar_height/2 + 0.072}" rpy="0.0 0.0 0.0"/>
         </xacro:property>
         <joint name="lidar_joint" type="fixed">
