Commit message: 23/6 commit. Localization MCL ran properly.

File: mecabot_description/urdf/include/common_macros.xacro (robot description, xacro)
@@ -23,5 +23,5 @@
     <!--~~~~~~~~~~ Layer and chassis properties ~~~~~~~~~~-->
     <xacro:property name="layer_l" value="0.255"/>
-    <xacro:property name="layer_w" value="0.15"/>
+    <xacro:property name="layer_w" value="0.148"/>
     <xacro:property name="layer_h" value="0.002"/>
     <xacro:property name="layer_mass" value="1.0"/>
@@ -52,5 +52,5 @@
     <!--~~~~~~~~~~ LiDAR properties ~~~~~~~~~~-->
     <xacro:property name="lidar_radius" value="0.035"/>
-    <xacro:property name="lidar_height" value="0.03"/>
+    <xacro:property name="lidar_height" value="0.075"/>
     <xacro:property name="lidar_mass" value="0.29"/>
 </robot>

File: mecabot_description/urdf/mecabot_core.xacro (robot description, xacro)
@@ -29,5 +29,5 @@
     <xacro:lidar parent="upper_layer"/>
     <!--~~~~~~~~~~ IMU ~~~~~~~~~~-->
-    <xacro:imu parent="base"/>
+    <xacro:imu parent="upper_layer"/>
     <!--~~~~~~~~~~ Extra simulation components (if use Gazebo). Change condition to False when run on real robot  ~~~~~~~~~~-->
     <xacro:if value="$(arg use_simulation)">

File: mecabot_description/urdf/sensors/imu.xacro (robot description, xacro)
@@ -3,5 +3,5 @@
     <xacro:macro name="imu" params="parent">
         <joint name="imu_joint" type="fixed">
-            <origin xyz="0.0 0.0 0.0" rpy="0.0 0.0 0.0"/>
+            <origin xyz="-0.1065 0.0 0.0" rpy="0.0 0.0 0.0"/>
             <parent link="${parent}_link"/>
             <child link="imu_frame"/>
